File: clock2.kicad_pcb (KiCad board)
At the start: 2 copper layers, 55 x 40 mm, 37 parts, among them CN1 PJ-327A 5JJ, CN2 PJ-327A 5JJ, SW1 SSSS811101, U1 NE555D, U2 NE555D, U3 TC-6615-9.0-160G, U4 NE555D, U5 XL74LS04, U6 XL74LS08, U7 XL74LS32, U8 RM063-105(1M)

Commit message: use the switching capability of the headphone jack to default the HALT signal to LOW. use resistor to prevent input HALT short to ground before contact breaks
Connections:
- CN2 pad 5: unconnected-(CN2-Pad5) -> GND
Changed lines of the file:
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@@
 	(net 55 "Net-(R2-Pad2)")
 	(net 56 "unconnected-(U8-Pad3)")
-	(net 57 "unconnected-(CN2-Pad5)")
 	(footprint "Resistor_SMD:R_0805_2012Metric_Pad1.20x1.40mm_HandSolder"
 		(layer "F.Cu")
@@
 			(size 2 3.2)
 			(layers "F.Cu" "F.Mask" "F.Paste")
-			(net 57 "unconnected-(CN2-Pad5)")
+			(net 6 "GND")
 			(pinfunction "5")
-			(pintype "unspecified+no_connect")
+			(pintype "unspecified")
 		)
 		(embedded_fonts no)

Commit message: v1 finalized
Parts:
- added R11: 1k, easyeda2kicad:R0805, F.Cu at (46.5, 30.7)
- C1, C2, C3, C4, C5, C6: footprint Capacitor_SMD:C_0805_2012Metric_Pad1.18x1.45mm_HandSolder -> easyeda2kicad:C0805
- R1, R10, R2, R3, R4, R5, R6, R7, R8, R9: footprint Resistor_SMD:R_0805_2012Metric_Pad1.20x1.40mm_HandSolder -> easyeda2kicad:R0805
- U1, U2, U4: footprint Package_SO:SOIC-8_3.9x4.9mm_P1.27mm -> easyeda2kicad:SOIC-8_L4.9-W3.9-P1.27-LS6.0-BL
- moved U5 18.8 mm to (19.5, 13.7), turned to 90 degrees
- moved U7 11.4 mm to (40.1, 13.5), turned to 0 degrees
- moved U6 10.2 mm to (29.2, 13.7)
- moved R5 4.66 mm to (30.7, 20.8), turned to 0 degrees
- moved C5 3.79 mm to (36.8, 24.1), turned to 180 degrees
- moved C4 3.69 mm to (36.8, 20.8), turned to 180 degrees
- moved DC1 2.26 mm to (10.5, 29.1)
- moved R4 1.68 mm to (37.1, 29.2), turned to 90 degrees
- moved R2 1.31 mm to (16.7, 30.7)
- moved C2 1.30 mm to (16.8, 24.6), turned to 180 degrees
- moved R1 1.25 mm to (16.8, 28.4), turned to 180 degrees
- moved U4 1.19 mm to (24.1, 22.9)
- moved REF** 0.79 mm to (46.0, 13.0)
- moved U1 0.69 mm to (23.1, 31.8), turned to 0 degrees
- moved C3 0.05 mm to (24.3, 37.6), turned to 0 degrees
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Connections:
- C1 pad 1: GND -> twosix
- C1 pad 2: twosix -> GND
- C2 pad 1: +5V -> GND
- C2 pad 2: GND -> +5V
- C3 pad 1: five -> GND
- C3 pad 2: GND -> five
- C4 pad 1: dis2 -> GND
- C4 pad 2: GND -> dis2
- C5 pad 1: five2 -> GND
- C5 pad 2: GND -> five2
- C6 pad 1: five3 -> GND
- C6 pad 2: GND -> five3
- CN2 pad 5: GND -> Net-(CN2-Pad5)
- R1 pad 1: +5V -> dis
- R1 pad 2: dis -> +5V
- R10 pad 1: GND -> Net-(D4-K)
- R10 pad 2: Net-(D4-K) -> GND
- R3 pad 1: GND -> Net-(D1-K)
- R3 pad 2: Net-(D1-K) -> GND
- R4 pad 1: +5V -> button
- R4 pad 2: button -> +5V
- R5 pad 1: dis2 -> +5V
- R5 pad 2: +5V -> dis2
- R6 pad 1: +5V -> switch
- R6 pad 2: switch -> +5V
- R7 pad 1: +5V -> switch2
- R7 pad 2: switch2 -> +5V
- R8 pad 1: GND -> Net-(D2-K)
- R8 pad 2: Net-(D2-K) -> GND
- R9 pad 1: GND -> Net-(D3-K)
- R9 pad 2: Net-(D3-K) -> GND
- U5 pad 3: unconnected-(U5-2A-Pad3) -> halt
- U5 pad 4: unconnected-(U5-2Y-Pad4) -> haltbar
- U5 pad 8: haltbar -> unconnected-(U5-4Y-Pad8)
- U5 pad 9: halt -> unconnected-(U5-4A-Pad9)
Routing:
- net GND: track 182.1 -> 209.8 mm, vias 1 -> 0
- net haltbar: track 27.9 -> 4.78 mm
- net halt: track 15.4 -> 36.7 mm
- net not1: track 30.5 -> 11.1 mm, vias 2 -> 0
- net realout: track 28.1 -> 45.0 mm
- net twosix: track 41.7 -> 27.2 mm, vias 1 -> 0
- net switch2: track 31.1 -> 22.2 mm
- net +5V: track 98.2 -> 89.6 mm, vias 3 -> 2
- net five3: track 4.58 -> 12.8 mm
- net and2: track 15.3 -> 8.48 mm
- net Net-(CN2-Pad5): track 0.00 -> 6.44 mm
- net out2: track 35.2 -> 29.2 mm
- net out: track 34.4 -> 40.0 mm
- net switch: track 27.6 -> 22.3 mm, vias 3 -> 2
- net and1: track 10.8 -> 5.70 mm
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Other:
- board text added: "@the_runofff"
